File: Hardware/_autosave-untitled.kicad_sch (KiCad schematic)
At the start: 14 parts, among them J1 Conn_02x05_Odd_Even, J2 USB_C_Receptacle_USB2.0_14P, SW1 SW_Push, U1 STM32F446RET6TR

Commit message: Routed USB-C components
Connections:
- net +3V3 is gone; now on net VCC: J1.7 (Pin_7)
- net +5V: now reaches J2.A4 (VBUS), J2.A9 (VBUS), J2.B4 (VBUS), J2.B9 (VBUS)
- net USB_DP: now reaches J2.A6 (D+)
- net USB_DP: now also J2.B6 (D+)
- net USB_DM: now reaches J2.A7 (D-)
- net USB_DM: now also J2.B7 (D-)
