File: Hardware/SD_Card.kicad_sch (KiCad schematic)
At the start: 3 parts, among them J6 DM3AT-SF-PEJM5

Commit message: Added hierarchal labels to main STM sheet and wired connections to SD card module
Connections:
- net CS renamed SD_CS
- net GPIO renamed SWA
Changed lines of the file:
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@@
 		)
 	)
-	(hierarchical_label "CS"
+	(hierarchical_label "SD_CS"
 		(shape input)
 		(at 99.06 88.9 180)
@@
 		)
 	)
-	(hierarchical_label "GPIO"
+	(hierarchical_label "SWA"
 		(shape input)
 		(at 123.19 99.06 180)

Commit message: Updated: ERC fixes
Connections:
- no-connect marks 0 -> 2
Changed lines of the file:
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@@
 		(color 0 0 0 0)
+	)
+	(no_connect
+		(at 125.73 83.82)
+	)
+	(no_connect
+		(at 125.73 86.36)
 	)
 	(wire
@@
 	(wire
 		(pts
+			(xy 123.19 93.98) (xy 125.73 93.98)
+		)
+		(stroke
+			(width 0)
+			(type default)
+		)
+	)
+	(wire
+		(pts
 			(xy 161.29 81.28) (xy 161.29 82.55)
 		)
@@
 		)
 		(stroke
-			(width 0)
-			(type default)
-		)
-	)
-	(wire
-		(pts
-			(xy 123.19 93.98) (xy 125.73 93.98)
-		)
-		(stroke
