File: Hardware/untitled.kicad_sch (KiCad schematic)
At the start: 14 parts, among them J1 Conn_02x05_Odd_Even, J2 USB_C_Receptacle_USB2.0_14P, SW1 SW_Push, U1 STM32F446RET6TR

Commit message: Added hierarchal sheets for the IMU and USB connectors. FInalized the design of USB and ESD protection
Parts:
- removed J2: USB_C_Receptacle_USB2.0_14P, symbol Connector:USB_C_Receptacle_USB2.0_14P
- removed R2, R3: 5.1kΩ, symbol Device:R
- added J5: Conn_01x04_Pin, symbol Connector:Conn_01x04_Pin
Connections:
- net VCC is gone; now on net +3V3: C1.1, C2.1, C3.1, C4.1, C5.1, U1.1 (VBAT), U1.13 (VDDA/VREF+), U1.19 (VDD), U1.32 (VDD), U1.48 (VDD), U1.64 (VDD)
- net +3V3: now also J5.1 (Pin_1)
- net GND: now also J5.4 (Pin_4)
- net SPI1_SCK: now reaches U1.21 (PA5)
- net SPI1_MISO: now reaches U1.22 (PA6)
- net SPI1_MOSI: now reaches U1.23 (PA7)
- net IMU_CS: now reaches U1.41 (PA8)
- net USB_DM: now reaches U1.44 (PA11)
- net USB_DP: now reaches U1.45 (PA12)
- new net GPS_RX: J5.2 (Pin_2)
- new net GPS_TX: J5.3 (Pin_3)
Other:
- note added: "GPS Connector"
- note added: "Stated on the datasheet that these were the pins for SWD configuration"
- moved on the sheet: C5, C6, C7, J1, R1, SW1, U1A, U1B

Commit message: Added hierarchal labels to main STM sheet and wired connections to SD card module
Connections:
- net SPI2_MISO: now reaches U1.10 (PC2)
- net SPI2_MOSI: now reaches U1.11 (PC3)
- net SPI2_SCK: now reaches U1.29 (PB10)
Other:
- moved on the sheet: C5, C6, U1B

Commit message: Updated: ERC fixes
Connections:
- net GPS_RX: now also U1.14 (PA0)
- net GPS_TX: now also U1.15 (PA1)
- net IMU_INT: now also U1.42 (PA9)
- net SD_CS: now also U1.61 (PB8)
- net SWA: now also U1.62 (PB9)
- no-connect marks 0 -> 39
Changed lines of the file:
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@@
 		(color 0 0 0 0)
 	)
+	(no_connect
+		(at 76.2 157.48)
+	)
+	(no_connect
+		(at 142.24 101.6)
+	)
+	(no_connect
+		(at 76.2 88.9)
+	)
+	(no_connect
+		(at 142.24 116.84)
+	)
+	(no_connect
+		(at 76.2 86.36)
+	)
+	(no_connect
+		(at 142.24 106.68)
+	)
+	(no_connect
+		(at 142.24 93.98)
+	)
+	(no_connect
+		(at 76.2 134.62)
+	)
+	(no_connect
+		(at 76.2 127)
+	)
+	(no_connect
+		(at 76.2 154.94)
+	)
+	(no_connect
+		(at 76.2 121.92)
+	)
+	(no_connect
+		(at 76.2 132.08)
+	)
+	(no_connect
+		(at 142.24 81.28)
+	)
+	(no_connect
+		(at 142.24 129.54)
+	)
+	(no_connect
+		(at 76.2 139.7)
+	)
+	(no_connect
+		(at 142.24 121.92)
+	)
+	(no_connect
+		(at 195.58 33.02)
+	)
+	(no_connect
+		(at 142.24 104.14)
+	)
+	(no_connect
+		(at 142.24 99.06)
+	)
+	(no_connect
+		(at 76.2 104.14)
+	)
+	(no_connect
+		(at 182.88 27.94)
+	)
+	(no_connect
+		(at 76.2 129.54)
+	)
+	(no_connect
+		(at 142.24 111.76)
+	)
+	(no_connect
+		(at 182.88 30.48)
+	)
+	(no_connect
+		(at 76.2 124.46)
+	)
+	(no_connect
+		(at 142.24 114.3)
+	)
+	(no_connect
+		(at 142.24 88.9)
+	)
+	(no_connect
+		(at 182.88 35.56)
+	)
+	(no_connect
+		(at 76.2 137.16)
+	)
+	(no_connect
+		(at 76.2 149.86)
+	)
+	(no_connect
+		(at 142.24 127)
+	)
+	(no_connect
+		(at 142.24 96.52)
+	)
+	(no_connect
+		(at 142.24 78.74)
+	)
+	(no_connect
+		(at 76.2 116.84)
+	)
+	(no_connect
+		(at 142.24 109.22)
+	)
+	(no_connect
+		(at 76.2 83.82)
+	)
+	(no_connect
+		(at 76.2 152.4)
+	)
+	(no_connect
+		(at 142.24 91.44)
+	)
+	(no_connect
+		(at 182.88 25.4)
+	)
 	(wire
 		(pts
@@
 	(wire
 		(pts
+			(xy 74.93 101.6) (xy 76.2 101.6)
+		)
+		(stroke
+			(width 0)
+			(type default)
+		)
+	)
+	(wire
+		(pts
 			(xy 186.69 81.28) (xy 190.5 81.28)
 		)
@@
 		)
 	)
+	(wire
+		(pts
+			(xy 73.66 78.74) (xy 76.2 78.74)
+		)
+		(stroke
+			(width 0)
+			(type default)
+		)
+	)
 	(bus
 		(pts
@@
 	(wire
 		(pts
+			(xy 73.66 81.28) (xy 76.2 81.28)
+		)
+		(stroke
+			(width 0)
+			(type default)
+		)
+	)
+	(wire
+		(pts
 			(xy 227.33 33.02) (xy 240.03 33.02)
 		)
@@
 	(wire
 		(pts
+			(xy 72.39 142.24) (xy 76.2 142.24)
+		)
+		(stroke
+			(width 0)
+			(type default)
+		)
+	)
+	(wire
+		(pts
 			(xy 73.66 106.68) (xy 76.2 106.68)
 		)
@@
 		(pts
 			(xy 262.89 71.12) (xy 262.89 68.58)
+		)
+		(stroke
+			(width 0)
+			(type default)
+		)
+	)
+	(wire
+		(pts
+			(xy 72.39 144.78) (xy 76.2 144.78)
 		)
 		(stroke
@@
 		)
 	)
+	(global_label "GPS_RX"
+		(shape input)
+		(at 73.66 78.74 180)
+		(fields_autoplaced yes)
+		(effects
+			(font
+				(size 1.27 1.27)
+			)
+			(justify right)
+		)
+		(property "Intersheetrefs" "${INTERSHEET_REFS}"
+			(at 63.4782 78.74 0)
+			(effects
+				(font
+					(size 1.27 1.27)
+				)
+				(justify right)
+				(hide yes)
+			)
+		)
+	)
 	(global_label "SWDIO"
 		(shape input)
@@
 		)
 	)
+	(global_label "GPS_TX"
+		(shape input)
+		(at 73.66 81.28 180)
+		(fields_autoplaced yes)
+		(effects
+			(font
+				(size 1.27 1.27)
+			)
+			(justify right)
+		)
+		(property "Intersheetrefs" "${INTERSHEET_REFS}"
+			(at 63.7806 81.28 0)
+			(effects
+				(font
+					(size 1.27 1.27)
+				)
+				(justify right)
+				(hide yes)
+			)
+		)
+	)
 	(hierarchical_label "SPI1_MISO"
 		(shape input)
@@
 	(hierarchical_label "SWA"
 		(shape input)
-		(at 39.37 146.05 180)
+		(at 72.39 144.78 180)
 		(effects
 			(font
@@
 	(hierarchical_label "SD_CS"
 		(shape input)
-		(at 39.37 143.51 180)
+		(at 72.39 142.24 180)
 		(effects
 			(font
@@
 	(hierarchical_label "IMU_INT"
 		(shape input)
-		(at 49.53 102.87 180)
-		(effects
-			(font
+		(at 74.93 101.6 180)
+		(effects
+			(font
